Commit message: 調整

File: my_robo_description/urdf/my_robo.urdf.xacro (robot description, xacro)
@@ -17,4 +17,9 @@
   <!---->
   <!---->
+  <link name="world"/>
+  <joint name="fixed" type="fixed">
+    <parent link="world"/>
+    <child link="base_link"/>
+  </joint>
   <link name="base_link"/>
   <link name="d435_link">
@@ -41,4 +46,14 @@
     <child link="d435_link" />
   </joint>
+  <link name="d435_link_optical"/>
+  <joint name="d435_link_to_d435_link_optical_joint" type="fixed">
+    <!-- these values have to be these values otherwise the gazebo camera
+        image won't be aligned properly with the frame it is supposedly
+        originating from -->
+    <!--https://answers.ros.org/question/232534/gazebo-camera-frame-is-inconsistent-with-rviz-opencv-convention/?answer=232562#post-id-232562-->
+    <origin xyz="0 0 0" rpy="${-pi/2} 0 ${-pi/2}"/>
+    <parent link="d435_link"/>
+    <child link="d435_link_optical"/>
+  </joint>
   <!--  gazebo-->
   <gazebo>
@@ -59,5 +74,5 @@
         <clip>
           <near>0.01</near>
-          <far>12</far>
+          <far>30</far>
         </clip>
       </camera>
@@ -71,6 +86,7 @@
         <depthImageCameraInfoTopicName>d435/depth/camera_info</depthImageCameraInfoTopicName>
         <pointCloudTopicName>d435/depth/points</pointCloudTopicName>
-        <frameName>d435_link</frameName>
-        <pointCloudCutoff>0.5</pointCloudCutoff>
+        <frameName>d435_link_optical</frameName>
+        <pointCloudCutoff>0.01</pointCloudCutoff>
+        <pointCloudCutoffMax>15.0</pointCloudCutoffMax>
         <distortionK1>0</distortionK1>
         <distortionK2>0</distortionK2>
